Commit message: person detection completed

File: person_follower_sim/urdf/mr_robot.xacro (robot description, xacro)
@@ -116,5 +116,5 @@
 	</link>
 	<joint name="kinect_camera_joint" type="fixed">
-			<origin rpy="0 0 0" xyz="0.15 -0.001759 0.073682"/>
+			<origin rpy="0 ${-pi/8} 0" xyz="0.15 -0.001759 0.073682"/>
 			<parent link="base_link"/>
 			<child link="kinect_camera"/>

Commit message: improved pid controller

File: person_follower_sim/urdf/mr_robot.xacro (robot description, xacro)
@@ -98,5 +98,5 @@
 	<link name="kinect_camera">
 		<collision>
-		  <origin xyz="0 0 0" rpy="0 0 0" />
+		  <origin xyz="0 0 0" rpy="0 1.2 0" />
 		<geometry>
 			<box size="0.07 0.3 0.09"/>
